File: DataLogger/DataLogger.kicad_sch (KiCad schematic)
At the start: 25 parts, among them U1 24LC1025, U2 24LC1025, U3 DS1337, U4 ATMEGA328P-AU, Y1 32.768 KHz, Y2 16MHz

Commit message: finished eeschema
Parts:
- U3: footprint DS1337:DIP794W47P254L991H457Q8 -> Package_SO:SOIC-8_3.9x4.9mm_P1.27mm
- U4: footprint ATMEGA328P-AU:QFP80P900X900X120-32N -> Package_QFP:TQFP-32_7x7mm_P0.8mm
Connections:
- net SCK: now also R3.2, R7.2, U1.6 (SCL), U2.6 (SCL), U3.6 (SCL), U4.17 (PB5), U4.28 (PC5)
- net SDA: now also R4.2, U1.5 (SDA), U2.5 (SDA), U3.5 (SDA), U4.27 (PC4)
- net RESET: now reaches R1.2, U4.29 (PC6/~{RESET})
- net D3: now reaches U4.1 (PD3)
- net D6: now reaches U4.10 (PD6)
- net D7: now reaches U4.11 (PD7)
- net MOSI: now reaches U4.15 (PB3)
- net MISO: now reaches U4.16 (PB4)
- net D4: now reaches U4.2 (PD4)
- net RX: now reaches U4.30 (PD0)
- net TX: now reaches U4.31 (PD1)
- net D2: now reaches U4.32 (PD2)
- net D5: now reaches U4.9 (PD5)
- no-connect marks 0 -> 10
Other:
- sheet Conn renamed CONN
- sheet CONN ports: added D2, D3, D4, D5, D6, D7, D8, GND, MISO, MOSI, RESET, RX, SCK, SDA, TX, VCC; removed none
- moved on the sheet: R1, R3, R4, U1, U2

Commit message: began pcbnew
Other:
- moved on the sheet: BT1, C2, C3, C4, C5, D1, D2, R1, R2, R3, R4, R7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
