File: DataLogger/DataLogger.kicad_pcb (KiCad board)
At the start: 2 copper layers, 29 parts, among them J1 Conn_01x04_Pin, J2 Conn_01x04_Pin, J3 Conn_01x09_Pin, J4 Conn_02x03_Odd_Even, U1 24LC1025, U2 24LC1025, U3 DS1337, U4 ATMEGA328P-AU, Y1 32.768 KHz, Y2 16MHz

Commit message: began pcbnew
Parts:
- moved U4 50.6 mm to (217.3, 106.6)
- moved J3 22.7 mm to (206.4, 84.0), turned to 90 degrees
- moved J4 7.70 mm to (233.5, 116.0), turned to 180 degrees
Changed lines of the file:
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@@
 	(footprint "Connector_PinHeader_2.54mm:PinHeader_1x09_P2.54mm_Vertical"
 		(layer "F.Cu")
-		(at 216.5 104.3)
+		(at 206.38 84 90)
 		(descr "Through hole straight pin header, 1x09, 2.54mm pitch, single row")
 		(tags "Through hole pin header THT 1x09 2.54mm single row")
 		(property "Reference" "J3"
-			(at 0 -2.38 0)
+			(at 0 -2.38 90)
 			(layer "F.SilkS")
 			(effects
@@
 		)
 		(property "Value" "Conn_01x09_Pin"
-			(at 3 11.78 90)
+			(at 3 11.78 0)
 			(layer "F.Fab")
 			(effects
@@
 		)
 		(property "Datasheet" ""
-			(at 0 0 0)
+			(at 0 0 90)
 			(layer "F.Fab")
 			(hide yes)
@@
 		)
 		(property "Description" "Generic connector, single row, 01x09, script generated"
-			(at 0 0 0)
+			(at 0 0 90)
 			(layer "F.Fab")
 			(hide yes)
@@
 		)
 		(property "KiLib_Generator" "connector/pin_header_socket"
-			(at 0 0 0)
+			(at 0 0 90)
 			(layer "F.SilkS")
 			(hide yes)
@@
 		)
 		(property "Purpose" "GPIO "
-			(at 0 0 0)
+			(at 0 0 90)
 			(unlocked yes)
 			(layer "F.Fab")
@@
 		)
 		(fp_line
-			(start -1.38 1.27)
-			(end -1.38 21.7)
+			(start 1.38 1.27)
+			(end 1.38 21.7)
 			(stroke
 				(width 0.12)
@@
 		)
 		(fp_line
-			(start -1.38 21.7)
-			(end 1.38 21.7)
+			(start -1.38 1.27)
+			(end -1.38 21.7)
 			(stroke
 				(width 0.12)
@@
 		)
 		(fp_line
-			(start 1.38 1.27)
+			(start -1.38 21.7)
 			(end 1.38 21.7)
 			(stroke
@@
 		)
 		(fp_line
-			(start -1.27 -0.635)
-			(end -0.635 -1.27)
+			(start 1.27 -1.27)
+			(end 1.27 21.59)
 			(stroke
 				(width 0.1)
@@
 		)
 		(fp_line
-			(start -1.27 21.59)
-			(end -1.27 -0.635)
+			(start -0.635 -1.27)
+			(end 1.27 -1.27)
 			(stroke
 				(width 0.1)
@@
 		)
 		(fp_line
-			(start -0.635 -1.27)
-			(end 1.27 -1.27)
+			(start -1.27 -0.635)
+			(end -0.635 -1.27)
 			(stroke
 				(width 0.1)
@@
 		)
 		(fp_line
-			(start 1.27 -1.27)
-			(end 1.27 21.59)
+			(start 1.27 21.59)
+			(end -1.27 21.59)
 			(stroke
 				(width 0.1)
@@
 		)
 		(fp_line
-			(start 1.27 21.59)
-			(end -1.27 21.59)
+			(start -1.27 21.59)
+			(end -1.27 -0.635)
 			(stroke
 				(width 0.1)
@@
 		)
 		(fp_text user "${REFERENCE}"
-			(at 0 10.16 90)
+			(at 0 10.16 0)
 			(layer "F.Fab")
 			(effects
@@
 		)
 		(pad "1" thru_hole rect
-			(at 0 0)
+			(at 0 0 90)
 			(size 1.7 1.7)
 			(drill 1)
@@
 		)
 		(pad "2" thru_hole circle
-			(at 0 2.54)
+			(at 0 2.54 90)
 			(size 1.7 1.7)
 			(drill 1)
@@
 		)
 		(pad "3" thru_hole circle
-			(at 0 5.08)
+			(at 0 5.08 90)
 			(size 1.7 1.7)
 			(drill 1)
@@
 		)
 		(pad "4" thru_hole circle
-			(at 0 7.62)
+			(at 0 7.62 90)
 			(size 1.7 1.7)
 			(drill 1)
@@
 		)
 		(pad "5" thru_hole circle
-			(at 0 10.16)
+			(at 0 10.16 90)
 			(size 1.7 1.7)
 			(drill 1)
@@
 		)
 		(pad "6" thru_hole circle
-			(at 0 12.7)
+			(at 0 12.7 90)
 			(size 1.7 1.7)
 			(drill 1)
@@
 		)
 		(pad "7" thru_hole circle
-			(at 0 15.24)
+			(at 0 15.24 90)
 			(size 1.7 1.7)
 			(drill 1)
@@
 		)
 		(pad "8" thru_hole circle
-			(at 0 17.78)
+			(at 0 17.78 90)
 			(size 1.7 1.7)
 			(drill 1)
@@
 		)
 		(pad "9" thru_hole circle
-			(at 0 20.32)
+			(at 0 20.32 90)
 			(size 1.7 1.7)
 			(drill 1)
@@
 	(footprint "Package_QFP:TQFP-32_7x7mm_P0.8mm"
 		(layer "F.Cu")
-		(at 168.125 118.235)
+		(at 217.3375 106.6)
 		(descr "TQFP, 32 Pin (JEDEC MS-026 variation ABA, https://www.jedec.org/document_search?search_api_views_fulltext=MS-026, https://ww1.microchip.com/downloads/en/PackagingSpec/00000049BZ.pdf#page=656)")
 		(tags "TQFP QFP")
@@
 	(footprint "Connector_PinHeader_2.54mm:PinHeader_2x03_P2.54mm_Vertical"
 		(layer "F.Cu")
-		(at 225.96 117.42)
+		(at 233.54 116.04 180)
 		(descr "Through hole straight pin header, 2x03, 2.54mm pitch, double rows")
 		(tags "Through hole pin header THT 2x03 2.54mm double row")
@@
 		)
 		(property "Purpose" "ICSP"
-			(at 0 0 0)
+			(at 0 0 180)
 			(unlocked yes)
 			(layer "F.Fab")
@@
 		(duplicate_pad_numbers_are_jumpers no)
 		(fp_line
-			(start -1.38 -1.38)
-			(end 0 -1.38)
+			(start 3.92 -1.38)
+			(end 3.92 6.46)
 			(stroke
 				(width 0.12)
@@
 		)
 		(fp_line
-			(start -1.38 0)
-			(end -1.38 -1.38)
+			(start 1.27 1.27)
+			(end 1.27 -1.38)
 			(stroke
 				(width 0.12)
@@
 		)
 		(fp_line
-			(start -1.38 1.27)
-			(end -1.38 6.46)
+			(start 1.27 -1.38)
+			(end 3.92 -1.38)
 			(stroke
 				(width 0.12)
@@
 		)
 		(fp_line
-			(start -1.38 1.27)
-			(end 1.27 1.27)
+			(start -1.38 6.46)
+			(end 3.92 6.46)
 			(stroke
 				(width 0.12)
@@
 		)
 		(fp_line
-			(start -1.38 6.46)
-			(end 3.92 6.46)
+			(start -1.38 1.27)
+			(end 1.27 1.27)
 			(stroke
 				(width 0.12)
@@
 		)
 		(fp_line
-			(start 1.27 -1.38)
-			(end 3.92 -1.38)
+			(start -1.38 1.27)
+			(end -1.38 6.46)
 			(stroke
 				(width 0.12)
@@
 		)
 		(fp_line
-			(start 1.27 1.27)
-			(end 1.27 -1.38)
+			(start -1.38 0)
+			(end -1.38 -1.38)
 			(stroke
 				(width 0.12)
@@
 		)
 		(fp_line
-			(start 3.92 -1.38)
-			(end 3.92 6.46)
+			(start -1.38 -1.38)
+			(end 0 -1.38)
 			(stroke
 				(width 0.12)
@@
 		)
 		(fp_line
-			(start -1.27 0)
-			(end 0 -1.27)
+			(start 3.81 6.35)
+			(end -1.27 6.35)
 			(stroke
 				(width 0.1)
@@
 		)
 		(fp_line
-			(start -1.27 6.35)
-			(end -1.27 0)
+			(start 3.81 -1.27)
+			(end 3.81 6.35)
 			(stroke
 				(width 0.1)
@@
 		)
 		(fp_line
-			(start 3.81 -1.27)
-			(end 3.81 6.35)
+			(start -1.27 6.35)
+			(end -1.27 0)
 			(stroke
 				(width 0.1)
@@
 		)
 		(fp_line
-			(start 3.81 6.35)
-			(end -1.27 6.35)
+			(start -1.27 0)
+			(end 0 -1.27)
 			(stroke
 				(width 0.1)
@@
 		)
 		(pad "1" thru_hole rect
-			(at 0 0)
+			(at 0 0 180)
 			(size 1.7 1.7)
 			(drill 1)
@@
 		)
 		(pad "2" thru_hole circle
-			(at 2.54 0)
+			(at 2.54 0 180)
 			(size 1.7 1.7)
 			(drill 1)
@@
 		)
 		(pad "3" thru_hole circle
-			(at 0 2.54)
+			(at 0 2.54 180)
 			(size 1.7 1.7)
 			(drill 1)
@@
 		)
 		(pad "4" thru_hole circle
-			(at 2.54 2.54)
+			(at 2.54 2.54 180)
 			(size 1.7 1.7)
 			(drill 1)
@@
 		)
 		(pad "5" thru_hole circle
-			(at 0 5.08)
+			(at 0 5.08 180)
 			(size 1.7 1.7)
 			(drill 1)
@@
 		)
 		(pad "6" thru_hole circle
-			(at 2.54 5.08)
+			(at 2.54 5.08 180)
 			(size 1.7 1.7)
 			(drill 1)

Commit message: /
Parts:
- removed BT1: Battery, Battery:BatteryHolder_Keystone_103_1x20mm
- removed C1: 0.1uF, Capacitor_SMD:C_1210_3225Metric
- removed C2, C3: 22pF, Capacitor_SMD:C_0201_0603Metric
- removed C4: 0.1uF, Capacitor_SMD:C_0201_0603Metric
- removed C5: 100nF, Capacitor_SMD:CP_Elec_4x3
- removed D1: LED, LED_SMD:LED_0201_0603Metric
- removed D2: LED, LED_SMD:LED_1210_3225Metric
- removed H1, H2, H3, H4: MountingHole, MountingHole:MountingHole_2.1mm
- removed J1, J2: Conn_01x04_Pin, Connector_PinHeader_2.54mm:PinHeader_1x04_P2.54mm_Vertical
- removed J3: Conn_01x09_Pin, Connector_PinHeader_2.54mm:PinHeader_1x09_P2.54mm_Vertical
- removed J4: Conn_02x03_Odd_Even, Connector_PinHeader_2.54mm:PinHeader_2x03_P2.54mm_Vertical
- removed R1, R5, R6: 10k, Resistor_SMD:R_0805_2012Metric
- removed R2, R7: 330, Resistor_SMD:R_0805_2012Metric
- removed R3, R4: 4.7k, Resistor_SMD:R_0805_2012Metric
- removed U1, U2: 24LC1025, Package_SO:SOIC-8_3.9x4.9mm_P1.27mm
- removed U3: DS1337, Package_SO:SOIC-8_3.9x4.9mm_P1.27mm
- removed U4: ATMEGA328P-AU, Package_QFP:TQFP-32_7x7mm_P0.8mm
- removed Y1: 32.768 KHz, Crystal:Crystal_SMD_5032-2Pin_5.0x3.2mm
- removed Y2: 16MHz, Crystal:Crystal_SMD_5032-2Pin_5.0x3.2mm

Commit message: added wiring
Parts:
- added BT1: Battery, Battery:BatteryHolder_Keystone_103_1x20mm, F.Cu at (150.5, 105.5)
- added C1: 0.1uF, Capacitor_SMD:C_1210_3225Metric, F.Cu at (120.0, 97.0)
- added C2: 22pF, Capacitor_SMD:C_0201_0603Metric, F.Cu at (122.3, 109.6)
- added C3: 22pF, Capacitor_SMD:C_0201_0603Metric, F.Cu at (118.7, 109.6)
- added C4: 0.1uF, Capacitor_SMD:C_0201_0603Metric, F.Cu at (139.5, 104.4)
- added C5: 100nF, Capacitor_SMD:CP_Elec_4x3, F.Cu at (142.5, 108.2)
- added D1: LED, LED_SMD:LED_0201_0603Metric, F.Cu at (151.0, 112.0)
- added D2: LED, LED_SMD:LED_1210_3225Metric, F.Cu at (152.5, 91.0)
- added H1: MountingHole, MountingHole:MountingHole_2.1mm, F.Cu at (105.0, 81.0)
- added H2: MountingHole, MountingHole:MountingHole_2.1mm, F.Cu at (173.0, 81.0)
- added H3: MountingHole, MountingHole:MountingHole_2.1mm, F.Cu at (102.5, 122.5)
- added H4: MountingHole, MountingHole:MountingHole_2.1mm, F.Cu at (175.0, 122.0)
- added J1: Conn_01x04_Pin, Connector_PinHeader_2.54mm:PinHeader_1x04_P2.54mm_Vertical, F.Cu at (120.0, 81.0)
- added J2: Conn_01x04_Pin, Connector_PinHeader_2.54mm:PinHeader_1x04_P2.54mm_Vertical, F.Cu at (148.0, 81.0)
- added J3: Conn_01x09_Pin, Connector_PinHeader_2.54mm:PinHeader_1x09_P2.54mm_Vertical, F.Cu at (106.0, 96.0)
- added J4: Conn_02x03_Odd_Even, Connector_PinHeader_2.54mm:PinHeader_2x03_P2.54mm_Vertical, F.Cu at (128.0, 116.0)
- added R1: 10k, Resistor_SMD:R_0805_2012Metric, F.Cu at (127.0, 96.5)
- added R2: 330, Resistor_SMD:R_0805_2012Metric, F.Cu at (148.0, 112.0)
- added R3: 4.7k, Resistor_SMD:R_0805_2012Metric, F.Cu at (130.0, 96.5)
- added R4: 4.7k, Resistor_SMD:R_0805_2012Metric, F.Cu at (133.2, 96.5)
- added R5: 10k, Resistor_SMD:R_0805_2012Metric, F.Cu at (139.0, 96.0)
- added R6: 10k, Resistor_SMD:R_0805_2012Metric, F.Cu at (145.5, 90.4)
- added R7: 330, Resistor_SMD:R_0805_2012Metric, F.Cu at (150.0, 97.0)
- added U1: 24LC1025, Package_SO:SOIC-8_3.9x4.9mm_P1.27mm, F.Cu at (115.0, 91.0)
- added U2: 24LC1025, Package_SO:SOIC-8_3.9x4.9mm_P1.27mm, F.Cu at (124.0, 91.0)
- added U3: DS1337, Package_SO:SOIC-8_3.9x4.9mm_P1.27mm, F.Cu at (139.0, 91.0)
- added U4: ATMEGA328P-AU, Package_QFP:TQFP-32_7x7mm_P0.8mm, F.Cu at (132.0, 104.0)
- added Y1: 32.768 KHz, Crystal:Crystal_SMD_5032-2Pin_5.0x3.2mm, F.Cu at (131.5, 91.0)
- added Y2: 16MHz, Crystal:Crystal_SMD_5032-2Pin_5.0x3.2mm, F.Cu at (120.5, 106.4)
Other:
- board outline added: 82 x 51 mm
